File: main.kicad_pcb (KiCad board)
At the start: 2 copper layers, 65 x 65 mm, 120 parts, among them J1 Jack-DC, J2 HIROSE_FH12-34S-0.5SVA, J3 Raspberry_Pi_2_3, SW1 SW_Push, SW2 SW_Push, SW3 SW_Push, SW4 SW_Push, U1 TPS56339, U2 TPS51397A, U3 SN74LVC8T245PW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

Commit message: almost routed
Parts:
- moved JP11 8.46 mm to (45.1, 31.3), turned to 180 degrees
- moved R24 5.43 mm to (36.0, 29.6), turned to 180 degrees
- moved C28 3.28 mm to (22.1, 1.77)
- moved C29 3.28 mm to (22.1, 3.35)
- moved C30 3.28 mm to (22.1, 4.92)
- moved C31 3.28 mm to (22.1, 6.50)
- moved C32 3.28 mm to (22.1, 8.07)
- moved C33 3.28 mm to (22.1, 9.65)
- moved C36 3.28 mm to (22.1, 11.2)
- moved C37 3.28 mm to (22.1, 12.8)
- moved C38 3.28 mm to (22.1, 14.4)
- moved C39 3.28 mm to (22.1, 16.1)
- moved C40 3.28 mm to (22.1, 17.6)
- moved C41 3.28 mm to (22.1, 19.2)
- moved R33 3.28 mm to (26.4, 9.65)
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Routing:
- net +5V: track 26.5 -> 122.2 mm, vias 2 -> 13
- net Net-(R28-Pad2): track 0.00 -> 82.2 mm
- net Net-(R25-Pad2): track 0.00 -> 69.1 mm
- net Net-(R22-Pad2): track 0.00 -> 68.2 mm
- net +3V3: track 0.00 -> 64.4 mm, vias 0 -> 8
- net Net-(R20-Pad2): track 0.00 -> 57.9 mm
- net GND: track 2.20 -> 45.0 mm, vias 36 -> 79
- net /ROW-LATCH: track 0.00 -> 25.2 mm, vias 0 -> 2
- net /LATCH: track 0.00 -> 25.0 mm, vias 0 -> 2
- net /ROW-BLANK: track 0.00 -> 24.3 mm, vias 0 -> 2
- net /nOUT-EN: track 0.00 -> 23.1 mm
- net /ROW-DATA: track 0.00 -> 20.7 mm
- net /BLUE-1: track 0.00 -> 19.2 mm
- net /GREEN-1: track 0.00 -> 19.0 mm
- net Net-(R45-Pad1): track 0.00 -> 18.8 mm
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- added copper zone on B.Cu, net +5V

Commit message: routed
Parts:
- moved D5 47.9 mm to (29.9, 20.4), turned to 180 degrees
- moved R11 47.3 mm to (29.9, 22.1), turned to 0 degrees
- moved D1 8.07 mm to (53.5, 63.2), turned to 0 degrees
- moved R4 6.33 mm to (53.5, 61.5), turned to 180 degrees
Connections:
- J3 pad 1: +3V3 -> /+3V3_LED
- J3 pad 22: Net-(J3-Pad22) -> /LED-STATUS
- J3 pad 3: /LED-STATUS -> Net-(J3-Pad3)
- R4 pad 2: +3V3 -> /+3V3_LED
Routing:
- net /LED-STATUS: track 0.00 -> 37.3 mm
- net Net-(J3-Pad7): track 0.00 -> 30.6 mm, vias 0 -> 1
- net /+3V3_LED: track 0.00 -> 9.58 mm
- net GND: track 45.0 -> 54.3 mm, vias 79 -> 136
- net +5V: track 122.2 -> 130.5 mm
- net +5VP: track 13.0 -> 19.3 mm, vias 15 -> 37
- net +24V: track 50.3 -> 53.9 mm
- net +3V3: track 64.4 -> 67.7 mm
- net Net-(D1-Pad2): track 0.00 -> 1.72 mm
- net Net-(D5-Pad2): track 0.00 -> 1.72 mm
- net Net-(D2-Pad2): track 0.00 -> 1.67 mm
- net Net-(D3-Pad2): track 0.00 -> 1.62 mm
- net Net-(D4-Pad2): track 0.00 -> 1.57 mm
- net Net-(R22-Pad2): track 68.2 -> 67.0 mm
- net Net-(R20-Pad2): track 57.9 -> 56.7 mm
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- added copper zone on B.Cu, net +5VP
- added copper zone on B.Cu, net GND
Other:
- net class supply_voltage added: clearance 0.2, trace_width 0.2, via_dia 0.6, via_drill 0.3
