File: main.sch (KiCad schematic (older format))
At the start: 120 parts, among them J1 Jack-DC, J2 HIROSE_FH12-34S-0.5SVA, J3 Raspberry_Pi_2_3, SW1 SW_Push, SW2 SW_Push, SW3 SW_Push, SW4 SW_Push, U1 TPS56339, U2 TPS51397A, U3 SN74LVC8T245PW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

Commit message: routed
Connections:
- net +3V3: no longer J3.1 (3V3), R4.2
- net LED-STATUS: now also J3.22 (GPIO25); no longer J3.3 (SDA/GPIO2)
- new net +3V3_LED: J3.1 (3V3), R4.2
Changed lines of the file:
@@
 ROW-DATA
 Wire Wire Line
-	10650 6850 10650 6900
-Wire Wire Line
-	10750 7300 10750 7100
-Wire Wire Line
-	10750 7100 10650 7100
-Connection ~ 10650 7100
-Wire Wire Line
-	10650 7100 10650 7300
+	10750 6850 10750 6900
 $Comp
 L power:+3V3 #PWR0118
 U 1 1 609C1DC1
-P 10650 6850
-F 0 "#PWR0118" H 10650 6700 50  0001 C CNN
-F 1 "+3V3" H 10665 7023 50  0000 C CNN
-F 2 "" H 10650 6850 50  0001 C CNN
-F 3 "" H 10650 6850 50  0001 C CNN
-	1    10650 6850
+P 10750 6850
+F 0 "#PWR0118" H 10750 6700 50  0001 C CNN
+F 1 "+3V3" H 10765 7023 50  0000 C CNN
+F 2 "" H 10750 6850 50  0001 C CNN
+F 3 "" H 10750 6850 50  0001 C CNN
+	1    10750 6850
 	1    0    0    -1
 $EndComp
@@
 Wire Wire Line
 	10900 1650 11100 1650
-Wire Wire Line
-	11400 1650 11650 1650
 $Comp
 L Device:R R6
@@
 Wire Wire Line
 	10150 2450 10150 2600
-$Comp
-L power:+3V3 #PWR0135
-U 1 1 60C145DD
-P 11650 1450
-F 0 "#PWR0135" H 11650 1300 50  0001 C CNN
-F 1 "+3V3" H 11665 1623 50  0000 C CNN
-F 2 "" H 11650 1450 50  0001 C CNN
-F 3 "" H 11650 1450 50  0001 C CNN
-	1    11650 1450
-	1    0    0    -1
-$EndComp
-Wire Wire Line
-	11650 1650 11650 1450
-Wire Wire Line
-	11850 1850 11850 1450
-Wire Wire Line
-	11400 1850 11850 1850
-Wire Wire Line
-	12050 2050 12050 1450
-Wire Wire Line
-	11400 2050 12050 2050
+Wire Wire Line
+	12200 1850 12200 1450
+Wire Wire Line
+	11400 1850 12200 1850
+Wire Wire Line
+	12400 2050 12400 1450
+Wire Wire Line
+	11400 2050 12400 2050
 $Comp
 L power:+5V #PWR0136
 U 1 1 60CC242A
-P 11850 1450
-F 0 "#PWR0136" H 11850 1300 50  0001 C CNN
-F 1 "+5V" H 11865 1623 50  0000 C CNN
-F 2 "" H 11850 1450 50  0001 C CNN
-F 3 "" H 11850 1450 50  0001 C CNN
-	1    11850 1450
+P 12200 1450
+F 0 "#PWR0136" H 12200 1300 50  0001 C CNN
+F 1 "+5V" H 12215 1623 50  0000 C CNN
+F 2 "" H 12200 1450 50  0001 C CNN
+F 3 "" H 12200 1450 50  0001 C CNN
+	1    12200 1450
 	1    0    0    -1
 $EndComp
@@
 L power:+5VP #PWR0137
 U 1 1 60CC8D6E
-P 12050 1450
-F 0 "#PWR0137" H 12050 1300 50  0001 C CNN
-F 1 "+5VP" H 12065 1623 50  0000 C CNN
-F 2 "" H 12050 1450 50  0001 C CNN
-F 3 "" H 12050 1450 50  0001 C CNN
-	1    12050 1450
-	1    0    0    -1
-$EndComp
-Wire Wire Line
-	12300 2250 12300 1450
-Wire Wire Line
-	11400 2250 12300 2250
+P 12400 1450
+F 0 "#PWR0137" H 12400 1300 50  0001 C CNN
+F 1 "+5VP" H 12415 1623 50  0000 C CNN
+F 2 "" H 12400 1450 50  0001 C CNN
+F 3 "" H 12400 1450 50  0001 C CNN
+	1    12400 1450
+	1    0    0    -1
+$EndComp
+Wire Wire Line
+	12650 2250 12650 1450
+Wire Wire Line
+	11400 2250 12650 2250
 $Comp
 L power:+24V #PWR0138
 U 1 1 60D143F0
-P 12300 1450
-F 0 "#PWR0138" H 12300 1300 50  0001 C CNN
-F 1 "+24V" H 12315 1623 50  0000 C CNN
-F 2 "" H 12300 1450 50  0001 C CNN
-F 3 "" H 12300 1450 50  0001 C CNN
-	1    12300 1450
+P 12650 1450
+F 0 "#PWR0138" H 12650 1300 50  0001 C CNN
+F 1 "+24V" H 12665 1623 50  0000 C CNN
+F 2 "" H 12650 1450 50  0001 C CNN
+F 3 "" H 12650 1450 50  0001 C CNN
+	1    12650 1450
 	1    0    0    -1
 $EndComp
 Text Label 11550 2450 0    50   ~ 0
 LED-STATUS
-Text Label 11950 8000 2    50   ~ 0
+Text Label 8850 9100 0    50   ~ 0
 LED-STATUS
 $Comp
@@
 	11500 6950 11500 6900
 Wire Wire Line
-	11500 6900 10650 6900
-Connection ~ 10650 6900
-Wire Wire Line
-	10650 6900 10650 7100
+	11500 6900 10750 6900
+Connection ~ 10750 6900
 $Comp
 L power:GND #PWR0139
@@
 	12700 8700 13900 8700
 Wire Wire Line
-	11350 8000 11950 8000
+	8850 9100 9750 9100
+Wire Wire Line
+	10750 6900 10750 7300
+Wire Wire Line
+	10650 7300 10650 6700
+Text Label 10650 6700 3    50   ~ 0
++3V3_LED
+Text Label 11950 1650 2    50   ~ 0
++3V3_LED
+Wire Wire Line
+	11400 1650 11950 1650
 $EndSCHEMATC
